File: electronics/_saved_vi_curve_tracer.sch (KiCad schematic (older format))
At the start: 28 parts, among them P1 CONN_01X05, P2 USB_OTG, P3 CONN_01X03, P4 CONN_01X03, U1 MCP6001, U2 pic24f08km202, U3 ft230x

Commit message: Made the schematic more closely resemble the rework performed.
Connections:
- net labels removed: HZ_OUT_0
- wire segments 138 -> 135
Other:
- moved on the sheet: R2, R3, R4, R5
Changed lines of the file:
@@
 Text GLabel 2900 3900 0    60   Output ~ 0
 LZ_OUT_0
-Text GLabel 2900 4200 0    60   Input ~ 0
-HZ_OUT_0
 Text GLabel 2900 4300 0    60   Input ~ 0
 HZ_OUT_1
@@
 L MCP6001 U1
 U 1 1 56B38849
-P 5750 6150
-F 0 "U1" H 5800 6350 50  0000 C CNN
-F 1 "MCP6001" H 5950 5950 50  0000 C CNN
-F 2 "kicad_pcb:SOT-23-5" H 5700 6250 50  0001 C CNN
-F 3 "" H 5800 6350 50  0000 C CNN
-	1    5750 6150
+P 5750 5550
+F 0 "U1" H 5800 5750 50  0000 C CNN
+F 1 "MCP6001" H 5950 5350 50  0000 C CNN
+F 2 "kicad_pcb:SOT-23-5" H 5700 5650 50  0001 C CNN
+F 3 "" H 5800 5750 50  0000 C CNN
+	1    5750 5550
 	-1   0    0    -1
 $EndComp
@@
 L GNDD #PWR020
 U 1 1 56B38CA4
-P 5850 6550
-F 0 "#PWR020" H 5850 6300 50  0001 C CNN
-F 1 "GNDD" H 5850 6400 50  0000 C CNN
-F 2 "" H 5850 6550 50  0000 C CNN
-F 3 "" H 5850 6550 50  0000 C CNN
-	1    5850 6550
+P 5850 5900
+F 0 "#PWR020" H 5850 5650 50  0001 C CNN
+F 1 "GNDD" H 5850 5750 50  0000 C CNN
+F 2 "" H 5850 5900 50  0000 C CNN
+F 3 "" H 5850 5900 50  0000 C CNN
+	1    5850 5900
 	1    0    0    -1
 $EndComp
@@
 L +5V #PWR021
 U 1 1 56B38ED1
-P 5850 5750
-F 0 "#PWR021" H 5850 5600 50  0001 C CNN
-F 1 "+5V" H 5850 5890 50  0000 C CNN
-F 2 "" H 5850 5750 50  0000 C CNN
-F 3 "" H 5850 5750 50  0000 C CNN
-	1    5850 5750
+P 5850 5150
+F 0 "#PWR021" H 5850 5000 50  0001 C CNN
+F 1 "+5V" H 5850 5290 50  0000 C CNN
+F 2 "" H 5850 5150 50  0000 C CNN
+F 3 "" H 5850 5150 50  0000 C CNN
+	1    5850 5150
 	1    0    0    -1
 $EndComp
@@
 L R R4
 U 1 1 56B3978E
-P 6950 6050
-F 0 "R4" V 7040 6060 50  0000 C CNN
-F 1 "2.67k" V 6952 6050 50  0000 C CNN
-F 2 "kicad_pcb:SM_0603" V 6880 6050 30  0001 C CNN
-F 3 "" H 6950 6050 30  0000 C CNN
-	1    6950 6050
+P 6900 5450
+F 0 "R4" V 6990 5460 50  0000 C CNN
+F 1 "2.67k" V 6902 5450 50  0000 C CNN
+F 2 "kicad_pcb:SM_0603" V 6830 5450 30  0001 C CNN
+F 3 "" H 6900 5450 30  0000 C CNN
+	1    6900 5450
 	0    1    1    0
 $EndComp
@@
 L R R5
 U 1 1 56B39824
-P 6950 6250
-F 0 "R5" V 7040 6260 50  0000 C CNN
-F 1 "2.67k" V 6952 6250 50  0000 C CNN
-F 2 "kicad_pcb:SM_0603" V 6880 6250 30  0001 C CNN
-F 3 "" H 6950 6250 30  0000 C CNN
-	1    6950 6250
+P 6900 5650
+F 0 "R5" V 6990 5660 50  0000 C CNN
+F 1 "2.67k" V 6902 5650 50  0000 C CNN
+F 2 "kicad_pcb:SM_0603" V 6830 5650 30  0001 C CNN
+F 3 "" H 6900 5650 30  0000 C CNN
+	1    6900 5650
 	0    1    1    0
 $EndComp
@@
 L R R3
 U 1 1 56B39AAD
-P 6400 5650
-F 0 "R3" V 6490 5660 50  0000 C CNN
-F 1 "24k" V 6402 5650 50  0000 C CNN
-F 2 "kicad_pcb:SM_0603" V 6330 5650 30  0001 C CNN
-F 3 "" H 6400 5650 30  0000 C CNN
-	1    6400 5650
+P 6400 4900
+F 0 "R3" V 6490 4910 50  0000 C CNN
+F 1 "24k" V 6402 4900 50  0000 C CNN
+F 2 "kicad_pcb:SM_0603" V 6330 4900 30  0001 C CNN
+F 3 "" H 6400 4900 30  0000 C CNN
+	1    6400 4900
 	-1   0    0    1
 $EndComp
@@
 L R R2
 U 1 1 56B39BF7
-P 5800 7050
-F 0 "R2" V 5890 7060 50  0000 C CNN
-F 1 "24k" V 5802 7050 50  0000 C CNN
-F 2 "kicad_pcb:SM_0603" V 5730 7050 30  0001 C CNN
-F 3 "" H 5800 7050 30  0000 C CNN
-	1    5800 7050
+P 5850 6300
+F 0 "R2" V 5940 6310 50  0000 C CNN
+F 1 "24k" V 5852 6300 50  0000 C CNN
+F 2 "kicad_pcb:SM_0603" V 5780 6300 30  0001 C CNN
+F 3 "" H 5850 6300 30  0000 C CNN
+	1    5850 6300
 	0    -1   -1   0
 $EndComp
 Text Notes 9350 4100 0    60   ~ 0
 Sense Resistor
-Text Notes 6550 5700 0    60   ~ 0
+Text Notes 6550 4950 0    60   ~ 0
 Use HZ_OUT_1 to set the reference\nfor the differential amplifier.  May move it\naround to increase the effective range.
 $Comp
@@
 	3450 1450 3450 1600
 Wire Wire Line
-	2900 4200 3150 4200
-Wire Wire Line
 	3150 4300 2900 4300
 Wire Wire Line
@@
 	9200 4350 9200 4450
 Wire Wire Line
-	9200 4450 9200 6250
+	9200 4450 9200 5650
 Wire Wire Line
 	9200 3300 9900 3300
@@
 	10050 3400 10250 3400
 Wire Wire Line
-	5300 7050 5550 7050
-Wire Wire Line
-	5300 4400 5300 6150
-Wire Wire Line
-	5300 6150 5300 7050
-Connection ~ 5300 6150
-Wire Wire Line
-	6050 7050 6400 7050
-Wire Wire Line
-	6400 7050 6400 6250
-Wire Wire Line
-	6050 6250 6400 6250
-Wire Wire Line
-	6400 6250 6700 6250
-Connection ~ 6400 6250
-Wire Wire Line
-	6400 5900 6400 6050
-Wire Wire Line
-	6050 6050 6400 6050
-Wire Wire Line
-	6400 6050 6700 6050
-Connection ~ 6400 6050
-Wire Wire Line
-	5850 6450 5850 6550
-Wire Wire Line
-	5850 5750 5850 5850
-Wire Wire Line
-	7500 6050 7500 3800
+	5300 6300 5600 6300
+Wire Wire Line
+	5300 4400 5300 5550
+Wire Wire Line
+	5300 5550 5300 6300
+Connection ~ 5300 5550
+Wire Wire Line
+	6100 6300 6400 6300
+Wire Wire Line
+	6400 6300 6400 5650
+Wire Wire Line
+	6050 5650 6400 5650
+Wire Wire Line
+	6400 5650 6650 5650
+Connection ~ 6400 5650
+Wire Wire Line
+	6400 5150 6400 5450
+Wire Wire Line
+	6050 5450 6400 5450
+Wire Wire Line
+	6400 5450 6650 5450
+Connection ~ 6400 5450
+Wire Wire Line
+	5850 5850 5850 5900
+Wire Wire Line
+	5850 5150 5850 5250
+Wire Wire Line
+	7500 5450 7500 3800
 Wire Wire Line
 	7500 3800 8650 3800
@@
 Connection ~ 9200 3800
 Connection ~ 9200 4450
-Wire Wire Line
-	6400 5200 6400 5400
 Wire Wire Line
 	6150 3200 9750 3200
@@
 	2900 3900 3150 3900
 Wire Wire Line
-	5300 6150 5450 6150
+	5300 5550 5450 5550
 Wire Wire Line
 	5300 4400 4250 4400
-Wire Wire Line
-	6400 5200 6400 3900
 Connection ~ 6400 3900
 Wire Wire Line
-	6400 5200 6400 5200
-Wire Wire Line
-	7200 6050 7500 6050
-Wire Wire Line
-	9200 6250 7200 6250
+	7150 5450 7500 5450
+Wire Wire Line
+	9200 5650 7150 5650
+Wire Wire Line
+	6400 4650 6400 3900
 $EndSCHEMATC
