File: electronics/_saved_vi_curve_tracer.sch (KiCad schematic (older format))
At the start: 50 parts, among them P1 CONN_01X05, P2 USB_OTG, P3 CONN_01X03, P4 CONN_01X03, U1 MCP6004, U2 pic24f08km202, U3 ft230x

Commit message: Added electronics files, nearly complete
Parts:
- added C19, C20, C21, C22: 1uF, kicad_pcb:SM_0603, symbol Csmall
- gave numbers to parts that had none: 3
Connections:
- net +5V: now also C19.1, C20.1, C21.1, C22.1
- net GNDD: now also C19.2, C20.2, C21.2, C22.2
Other:
- moved on the sheet: C16, C17, C18, C9
